Commit message: Update model

File: robots/pioneer3at.xacro (robot description, xacro)
@@ -18,5 +18,5 @@
 			<origin xyz="0 0 0.177" rpy="0 0 0"/>
 			<geometry name="pioneer_geom">
-				<mesh filename="package://p3at_tutorial/meshes/p3at_meshes/chassis.stl"/>
+				<mesh filename="package://fcr2017/meshes/p3at_meshes/chassis.stl"/>
 			</geometry>
 			<material name="ChassisRed">
@@ -27,5 +27,5 @@
 			<origin xyz="0 0 0.177" rpy="0 0 0"/>
 				<geometry>
-					<mesh filename="package://p3at_tutorial/meshes/p3at_meshes/chassis.stl"/>
+					<mesh filename="package://fcr2017/meshes/p3at_meshes/chassis.stl"/>
 				</geometry>
 		</collision>
@@ -61,5 +61,5 @@
 			<origin xyz="0 0 0" rpy="0 0 0"/>
 			<geometry name="pioneer_geom">
-				<mesh filename="package://p3at_tutorial/meshes/p3at_meshes/top.stl"/>
+				<mesh filename="package://fcr2017/meshes/p3at_meshes/top.stl"/>
 			</geometry>
 			<material name="TopBlack">
@@ -93,5 +93,5 @@
 			<origin xyz="0 0 0" rpy="0 0 0"/>
 			<geometry name="pioneer_geom">
-				<mesh filename="package://p3at_tutorial/meshes/p3at_meshes/front_sonar.stl"/>
+				<mesh filename="package://fcr2017/meshes/p3at_meshes/front_sonar.stl"/>
 			</geometry>
 			<material name="SonarYellow">
@@ -124,5 +124,5 @@
 			<origin xyz="0 0 0" rpy="0 0 0"/>
 			<geometry name="pioneer_geom">
-				<mesh filename="package://p3at_tutorial/meshes/p3at_meshes/back_sonar.stl"/>
+				<mesh filename="package://fcr2017/meshes/p3at_meshes/back_sonar.stl"/>
 			</geometry>
 			<material name="SonarYellow">
@@ -145,4 +145,60 @@
 		<child link="back_sonar"/>
 	</joint>
+<link name="back_sonar_fake">
+    <inertial>
+            <mass value="0.1"/>
+            <origin xyz="0 0 0"/>
+            <inertia ixx="1.0" ixy="0.0" ixz="0.0"
+                 iyy="1.0" iyz="0.0" izz="1.0"/>
+    </inertial>
+<!--     <visual name="base_visual">
+            <origin xyz="0 0 0" rpy="0 0 0"/>
+            <geometry name="pioneer_geom">
+                <mesh filename="package://fcr2017/meshes/p3at_meshes/back_sonar.stl"/>
+            </geometry>
+            <material name="SonarYellow">
+                <color rgba="0.715 0.583 0.210 1.0"/>
+            </material>
+        </visual>
+        <collision>
+            <origin xyz="0 0 0" rpy="0 0 0"/>
+            <geometry>
+                <box size="0 0 0"/>
+            </geometry>
+        </collision> -->
+</link>
+<joint name="base_back_sonar_joint" type="fixed">
+    <origin xyz="0 0 0" rpy="0 0 3.1415"/>
+    <parent link="back_sonar"/>
+    <child link="back_sonar_fake"/>
+</joint>
+<link name="imu">
+    <inertial>
+            <mass value="0.1"/>
+            <origin xyz="0 0 0"/>
+            <inertia ixx="1.0" ixy="0.0" ixz="0.0"
+                 iyy="1.0" iyz="0.0" izz="1.0"/>
+    </inertial>
+<!--     <visual name="base_visual">
+            <origin xyz="0 0 0" rpy="0 0 0"/>
+            <geometry name="pioneer_geom">
+                <mesh filename="package://fcr2017/meshes/p3at_meshes/back_sonar.stl"/>
+            </geometry>
+            <material name="SonarYellow">
+                <color rgba="0.715 0.583 0.210 1.0"/>
+            </material>
+        </visual>
+        <collision>
+            <origin xyz="0 0 0" rpy="0 0 0"/>
+            <geometry>
+                <box size="0 0 0"/>
+            </geometry>
+        </collision> -->
+</link>
+<joint name="imu_joint" type="fixed">
+    <origin xyz="0 0 0" rpy="3.1415 0 0"/>
+    <parent link="base_link"/>
+    <child link="imu"/>
+</joint>
 <!-- Front Axles + Wheels + Hubcaps -->
 <xacro:macro name="p3at_front" params="suffix reflect">
@@ -157,5 +213,5 @@
 		<origin xyz="0 0 0" rpy="0 0 0"/>
 		<geometry name="pioneer_geom">
-			<mesh filename="package://p3at_tutorial/meshes/p3at_meshes/axle.stl"/>
+			<mesh filename="package://fcr2017/meshes/p3at_meshes/axle.stl"/>
 		</geometry>
 		<material name="AxleGrey">
@@ -188,5 +244,5 @@
 		<origin xyz="0 0 0" rpy="0 0 0"/>
 		<geometry name="pioneer_geom">
-			<mesh filename="package://p3at_tutorial/meshes/p3at_meshes/${suffix}_hubcap.stl"/>
+			<mesh filename="package://fcr2017/meshes/p3at_meshes/${suffix}_hubcap.stl"/>
 		</geometry>
 		<material name="HubcapYellow">
@@ -219,5 +275,5 @@
 		<origin xyz="0 0 0" rpy="0 0 0"/>
 		<geometry name="pioneer_geom">
-			<mesh filename="package://p3at_tutorial/meshes/p3at_meshes/wheel.stl"/>
+			<mesh filename="package://fcr2017/meshes/p3at_meshes/wheel.stl"/>
 		</geometry>
 		<material name="WheelBlack">
@@ -228,5 +284,5 @@
 		<origin xyz="0 0 0" rpy="${-3.1415927/2} 0 0"/>
 		<geometry>
-	    <!--mesh filename="package://p3at_tutorial/meshes/p3at_meshes/wheel.stl"/-->
+	    <!--mesh filename="package://fcr2017/meshes/p3at_meshes/wheel.stl"/-->
 	    <cylinder radius="0.111" length="0.075"/>
 		</geometry>
@@ -256,5 +312,5 @@
 		<origin xyz="0 0 0" rpy="0 0 0"/>
 		<geometry name="pioneer_geom">
-			<mesh filename="package://p3at_tutorial/meshes/p3at_meshes/axle.stl"/>
+			<mesh filename="package://fcr2017/meshes/p3at_meshes/axle.stl"/>
 		</geometry>
 		<material name="AxleGrey">
@@ -265,5 +321,5 @@
 		<origin xyz="0 0 0" rpy="0 0 0"/>
 		<geometry>
-			<mesh filename="package://p3at_tutorial/meshes/p3at_meshes/axle.stl"/>
+			<mesh filename="package://fcr2017/meshes/p3at_meshes/axle.stl"/>
 		</geometry>
 	</collision>
@@ -287,5 +343,5 @@
 		<origin xyz="0 0 0" rpy="0 0 0"/>
 		<geometry name="pioneer_geom">
-			<mesh filename="package://p3at_tutorial/meshes/p3at_meshes/${suffix}_hubcap.stl"/>
+			<mesh filename="package://fcr2017/meshes/p3at_meshes/${suffix}_hubcap.stl"/>
 		</geometry>
 		<material name="HubcapYellow"/>
@@ -294,5 +350,5 @@
 		<origin xyz="0 0 0" rpy="0 0 0"/>
 		<geometry>
-			<mesh filename="package://p3at_tutorial/meshes/p3at_meshes/${suffix}_hubcap.stl"/>
+			<mesh filename="package://fcr2017/meshes/p3at_meshes/${suffix}_hubcap.stl"/>
 		</geometry>
 	</collision>
@@ -316,5 +372,5 @@
 		<origin xyz="0 0 0" rpy="0 0 0"/>
 		<geometry name="pioneer_geom">
-			<mesh filename="package://p3at_tutorial/meshes/p3at_meshes/wheel.stl"/>
+			<mesh filename="package://fcr2017/meshes/p3at_meshes/wheel.stl"/>
 		</geometry>
 		<material name="WheelBlack"/>
@@ -323,5 +379,5 @@
 		<origin xyz="0 0 0" rpy="${-3.1415927/2} 0 0"/>
 		<geometry>
-	    <!--mesh filename="package://p3at_tutorial/meshes/p3at_meshes/wheel.stl"/-->
+	    <!--mesh filename="package://fcr2017/meshes/p3at_meshes/wheel.stl"/-->
 	    <cylinder radius="0.111" length="0.075"/>
 		</geometry>
@@ -395,5 +451,5 @@
       <origin xyz="0 0 0" rpy="0 0 0"/>
       <geometry>
-        <mesh filename="package://p3at_tutorial/meshes/hokuyo1.dae"/>
+        <mesh filename="package://fcr2017/meshes/hokuyo1.dae"/>
       </geometry>
     </visual>
@@ -438,5 +494,97 @@
       </plugin>
     </sensor>
-  </gazebo>
+</gazebo>
+<gazebo reference="front_sonar">
+    <sensor type="ray" name="front_sonar_sensor">
+      <pose>0 0 0 0 0 0</pose>
+      <visualize>false</visualize>
+      <update_rate>25</update_rate>
+      <ray>
+        <scan>
+          <horizontal>
+            <samples>8</samples>
+            <resolution>1</resolution>
+            <min_angle>-1.570796</min_angle>
+            <max_angle>1.570796</max_angle>
+<!--             <samples>16</samples>
+            <resolution>1</resolution>
+            <min_angle>-1.919862</min_angle>
+            <max_angle>1.919862</max_angle> -->
+          </horizontal>
+        </scan>
+        <range>
+          <min>0.10</min>
+          <max>5.0</max>
+          <resolution>0.1</resolution>
+        </range>
+        <noise>
+          <type>gaussian</type>
+          <!-- Noise parameters based on published spec for Hokuyo laser
+               achieving "+-30mm" accuracy at range < 10m.  A mean of 0.0m and
+               stddev of 0.01m will put 99.7% of samples within 0.03m of the true
+               reading. -->
+          <mean>0.0</mean>
+          <stddev>0.1</stddev>
+        </noise>
+      </ray>
+      <plugin name="gazebo_ros_front_sonar_controller" filename="libgazebo_ros_laser.so">
+        <topicName>/front_sonar_raw</topicName>
+        <frameName>front_sonar</frameName>
+      </plugin>
+    </sensor>
+</gazebo>
+<gazebo reference="back_sonar_fake">
+    <sensor type="ray" name="back_sonar_sensor">
+      <pose>0 0 0 0 0 0</pose>
+      <visualize>false</visualize>
+      <update_rate>25</update_rate>
+      <ray>
+        <scan>
+          <horizontal>
+            <samples>8</samples>
+            <resolution>1</resolution>
+            <min_angle>-1.570796</min_angle>
+            <max_angle>1.570796</max_angle>
+<!--             <samples>16</samples>
+            <resolution>1</resolution>
+            <min_angle>-1.919862</min_angle>
+            <max_angle>1.919862</max_angle> -->
+          </horizontal>
+        </scan>
+        <range>
+          <min>0.10</min>
+          <max>5.0</max>
+          <resolution>0.1</resolution>
+        </range>
+        <noise>
+          <type>gaussian</type>
+          <!-- Noise parameters based on published spec for Hokuyo laser
+               achieving "+-30mm" accuracy at range < 10m.  A mean of 0.0m and
+               stddev of 0.01m will put 99.7% of samples within 0.03m of the true
+               reading. -->
+          <mean>0.0</mean>
+          <stddev>0.1</stddev>
+        </noise>
+      </ray>
+      <plugin name="gazebo_ros_back_sonar_controller" filename="libgazebo_ros_laser.so">
+        <topicName>/back_sonar_raw</topicName>
+        <frameName>back_sonar_fake</frameName>
+      </plugin>
+    </sensor>
+</gazebo>
+<gazebo>
+    <plugin name="imu_controller" filename="libhector_gazebo_ros_imu.so">
+        <robotNamespace>/</robotNamespace>
+        <updateRate>50.0</updateRate>
+        <bodyName>imu</bodyName>
+        <topicName>imu/data_raw</topicName>
+        <accelDrift>0.05 0.05 0.05</accelDrift>
+        <accelGaussianNoise>0.05 0.05 0.05</accelGaussianNoise>
+        <rateDrift>0.05 0.05 0.05 </rateDrift>
+        <rateGaussianNoise>0.05 0.05 0.05 </rateGaussianNoise>
+        <headingDrift>0.05</headingDrift>
+        <headingGaussianNoise>0.05</headingGaussianNoise>
+    </plugin>
+</gazebo>
 </xacro:macro>
 <xacro:p3at_front suffix="left" reflect="1"/>

Commit message: fix package name bug

File: robots/pioneer3at.xacro (robot description, xacro)
@@ -18,5 +18,5 @@
 			<origin xyz="0 0 0.177" rpy="0 0 0"/>
 			<geometry name="pioneer_geom">
-				<mesh filename="package://fcr2017/meshes/p3at_meshes/chassis.stl"/>
+				<mesh filename="package://p3at_tutorial/meshes/p3at_meshes/chassis.stl"/>
 			</geometry>
 			<material name="ChassisRed">
@@ -27,5 +27,5 @@
 			<origin xyz="0 0 0.177" rpy="0 0 0"/>
 				<geometry>
-					<mesh filename="package://fcr2017/meshes/p3at_meshes/chassis.stl"/>
+					<mesh filename="package://p3at_tutorial/meshes/p3at_meshes/chassis.stl"/>
 				</geometry>
 		</collision>
@@ -61,5 +61,5 @@
 			<origin xyz="0 0 0" rpy="0 0 0"/>
 			<geometry name="pioneer_geom">
-				<mesh filename="package://fcr2017/meshes/p3at_meshes/top.stl"/>
+				<mesh filename="package://p3at_tutorial/meshes/p3at_meshes/top.stl"/>
 			</geometry>
 			<material name="TopBlack">
@@ -93,5 +93,5 @@
 			<origin xyz="0 0 0" rpy="0 0 0"/>
 			<geometry name="pioneer_geom">
-				<mesh filename="package://fcr2017/meshes/p3at_meshes/front_sonar.stl"/>
+				<mesh filename="package://p3at_tutorial/meshes/p3at_meshes/front_sonar.stl"/>
 			</geometry>
 			<material name="SonarYellow">
@@ -124,5 +124,5 @@
 			<origin xyz="0 0 0" rpy="0 0 0"/>
 			<geometry name="pioneer_geom">
-				<mesh filename="package://fcr2017/meshes/p3at_meshes/back_sonar.stl"/>
+				<mesh filename="package://p3at_tutorial/meshes/p3at_meshes/back_sonar.stl"/>
 			</geometry>
 			<material name="SonarYellow">
@@ -155,5 +155,5 @@
             <origin xyz="0 0 0" rpy="0 0 0"/>
             <geometry name="pioneer_geom">
-                <mesh filename="package://fcr2017/meshes/p3at_meshes/back_sonar.stl"/>
+                <mesh filename="package://p3at_tutorial/meshes/p3at_meshes/back_sonar.stl"/>
             </geometry>
             <material name="SonarYellow">
@@ -183,5 +183,5 @@
             <origin xyz="0 0 0" rpy="0 0 0"/>
             <geometry name="pioneer_geom">
-                <mesh filename="package://fcr2017/meshes/p3at_meshes/back_sonar.stl"/>
+                <mesh filename="package://p3at_tutorial/meshes/p3at_meshes/back_sonar.stl"/>
             </geometry>
             <material name="SonarYellow">
@@ -213,5 +213,5 @@
 		<origin xyz="0 0 0" rpy="0 0 0"/>
 		<geometry name="pioneer_geom">
-			<mesh filename="package://fcr2017/meshes/p3at_meshes/axle.stl"/>
+			<mesh filename="package://p3at_tutorial/meshes/p3at_meshes/axle.stl"/>
 		</geometry>
 		<material name="AxleGrey">
@@ -244,5 +244,5 @@
 		<origin xyz="0 0 0" rpy="0 0 0"/>
 		<geometry name="pioneer_geom">
-			<mesh filename="package://fcr2017/meshes/p3at_meshes/${suffix}_hubcap.stl"/>
+			<mesh filename="package://p3at_tutorial/meshes/p3at_meshes/${suffix}_hubcap.stl"/>
 		</geometry>
 		<material name="HubcapYellow">
@@ -275,5 +275,5 @@
 		<origin xyz="0 0 0" rpy="0 0 0"/>
 		<geometry name="pioneer_geom">
-			<mesh filename="package://fcr2017/meshes/p3at_meshes/wheel.stl"/>
+			<mesh filename="package://p3at_tutorial/meshes/p3at_meshes/wheel.stl"/>
 		</geometry>
 		<material name="WheelBlack">
@@ -284,5 +284,5 @@
 		<origin xyz="0 0 0" rpy="${-3.1415927/2} 0 0"/>
 		<geometry>
-	    <!--mesh filename="package://fcr2017/meshes/p3at_meshes/wheel.stl"/-->
+	    <!--mesh filename="package://p3at_tutorial/meshes/p3at_meshes/wheel.stl"/-->
 	    <cylinder radius="0.111" length="0.075"/>
 		</geometry>
@@ -312,5 +312,5 @@
 		<origin xyz="0 0 0" rpy="0 0 0"/>
 		<geometry name="pioneer_geom">
-			<mesh filename="package://fcr2017/meshes/p3at_meshes/axle.stl"/>
+			<mesh filename="package://p3at_tutorial/meshes/p3at_meshes/axle.stl"/>
 		</geometry>
 		<material name="AxleGrey">
@@ -321,5 +321,5 @@
 		<origin xyz="0 0 0" rpy="0 0 0"/>
 		<geometry>
-			<mesh filename="package://fcr2017/meshes/p3at_meshes/axle.stl"/>
+			<mesh filename="package://p3at_tutorial/meshes/p3at_meshes/axle.stl"/>
 		</geometry>
 	</collision>
@@ -343,5 +343,5 @@
 		<origin xyz="0 0 0" rpy="0 0 0"/>
 		<geometry name="pioneer_geom">
-			<mesh filename="package://fcr2017/meshes/p3at_meshes/${suffix}_hubcap.stl"/>
+			<mesh filename="package://p3at_tutorial/meshes/p3at_meshes/${suffix}_hubcap.stl"/>
 		</geometry>
 		<material name="HubcapYellow"/>
@@ -350,5 +350,5 @@
 		<origin xyz="0 0 0" rpy="0 0 0"/>
 		<geometry>
-			<mesh filename="package://fcr2017/meshes/p3at_meshes/${suffix}_hubcap.stl"/>
+			<mesh filename="package://p3at_tutorial/meshes/p3at_meshes/${suffix}_hubcap.stl"/>
 		</geometry>
 	</collision>
@@ -372,5 +372,5 @@
 		<origin xyz="0 0 0" rpy="0 0 0"/>
 		<geometry name="pioneer_geom">
-			<mesh filename="package://fcr2017/meshes/p3at_meshes/wheel.stl"/>
+			<mesh filename="package://p3at_tutorial/meshes/p3at_meshes/wheel.stl"/>
 		</geometry>
 		<material name="WheelBlack"/>
@@ -379,5 +379,5 @@
 		<origin xyz="0 0 0" rpy="${-3.1415927/2} 0 0"/>
 		<geometry>
-	    <!--mesh filename="package://fcr2017/meshes/p3at_meshes/wheel.stl"/-->
+	    <!--mesh filename="package://p3at_tutorial/meshes/p3at_meshes/wheel.stl"/-->
 	    <cylinder radius="0.111" length="0.075"/>
 		</geometry>
@@ -451,5 +451,5 @@
       <origin xyz="0 0 0" rpy="0 0 0"/>
       <geometry>
-        <mesh filename="package://fcr2017/meshes/hokuyo1.dae"/>
+        <mesh filename="package://p3at_tutorial/meshes/hokuyo1.dae"/>
       </geometry>
     </visual>
