Commit message: Update xacro file for ros kinetic

File: robots/pioneer3at.xacro (robot description, xacro)
@@ -7,153 +7,91 @@
 >
 <!-- Chassis -->
-	<link name="base_link">
-		<inertial>
-			<mass value="10.0"/>
-			<origin xyz="0 0 0.177"/>
-			<inertia ixx="0.3338" ixy="0.0" ixz="0.0"
-				 iyy="0.4783" iyz="0.0"
-				 izz="0.3338"/>
-		</inertial>
-		<visual name="base_visual">
-			<origin xyz="0 0 0.177" rpy="0 0 0"/>
-			<geometry name="pioneer_geom">
-				<mesh filename="package://p3at_tutorial/meshes/p3at_meshes/chassis.stl"/>
-			</geometry>
-			<material name="ChassisRed">
-				<color rgba="0.851 0.0 0.0 1.0"/>
-			</material>
-		</visual>
-		<collision>
-			<origin xyz="0 0 0.177" rpy="0 0 0"/>
-				<geometry>
-					<mesh filename="package://p3at_tutorial/meshes/p3at_meshes/chassis.stl"/>
-				</geometry>
-		</collision>
-	</link>
-	<gazebo reference="base_link">
-		<material value="Gazebo/Red"/>
-	</gazebo>
+    <link name="base_link">
+        <inertial>
+            <mass value="10.0"/>
+            <origin xyz="0 0 0.177"/>
+            <inertia ixx="0.3338" ixy="0.0" ixz="0.0"
+                 iyy="0.4783" iyz="0.0"
+                 izz="0.3338"/>
+        </inertial>
+        <visual name="base_visual">
+            <origin xyz="0 0 0.177" rpy="0 0 0"/>
+            <geometry name="pioneer_geom">
+                <mesh filename="package://p3at_tutorial/meshes/p3at_meshes/chassis.dae"/>
+            </geometry>
+            <material name="ChassisRed">
+                <color rgba="0.851 0.0 0.0 1.0"/>
+            </material>
+        </visual>
+        <collision>
+            <origin xyz="0 0 0.177" rpy="0 0 0"/>
+                <geometry>
+                    <mesh filename="package://p3at_tutorial/meshes/p3at_meshes/chassis.dae"/>
+                </geometry>
+        </collision>
+    </link>
+    <gazebo reference="base_link">
+        <material value="Gazebo/Red"/>
+    </gazebo>
 <!--link name="odom">
 </link>
 <joint name="odom_base" type="floating">
-		<origin xyz="0 0 0" rpy="0 0 0"/>
-		<parent link="odom"/>
-		<child link="base_link"/>
-	</joint-->
+        <origin xyz="0 0 0" rpy="0 0 0"/>
+        <parent link="odom"/>
+        <child link="base_link"/>
+    </joint-->
 <!--<link name="map">
 </link-->
 <!--<joint name="map_odom" type="fixed">
-		<origin xyz="0 0 0" rpy="0 0 0"/>
-		<parent link="map"/>
-		<child link="odom"/>
-	</joint>
-	-->
+        <origin xyz="0 0 0" rpy="0 0 0"/>
+        <parent link="map"/>
+        <child link="odom"/>
+    </joint>
+    -->
 <!-- Top -->
-	<link name="top_plate">
-		<inertial>
-			<mass value="0.1"/>
-			<origin xyz="-0.025 0 -0.223"/>
-			<inertia ixx="1.0" ixy="0.0" ixz="0.0"
-				 iyy="1.0" iyz="0.0"
- 				izz="1.0"/>
-		</inertial>
-		<visual name="base_visual">
-			<origin xyz="0 0 0" rpy="0 0 0"/>
-			<geometry name="pioneer_geom">
-				<mesh filename="package://p3at_tutorial/meshes/p3at_meshes/top.stl"/>
-			</geometry>
-			<material name="TopBlack">
-					<color rgba="0.038 0.038 0.038 1.0"/>
-			</material>
-		</visual>
-		<collision>
-			<origin xyz="0 0 0" rpy="0 0 0"/>
-			<geometry>
-				<box size="0 0 0"/>
-			</geometry>
-		</collision>
-	</link>
-	<gazebo reference="top_plate">
-		<material value="Gazebo/Black"/>
-	</gazebo>
-	<joint name="base_top_joint" type="fixed">
-		<origin xyz="0.003 0 0.274" rpy="0 0 0"/>
-		<parent link="base_link"/>
-		<child link="top_plate"/>
-	</joint>
+    <link name="top_plate">
+        <inertial>
+            <mass value="0.1"/>
+            <origin xyz="-0.025 0 -0.223"/>
+            <inertia ixx="1.0" ixy="0.0" ixz="0.0"
+                 iyy="1.0" iyz="0.0"
+                izz="1.0"/>
+        </inertial>
+        <visual name="base_visual">
+            <origin xyz="0 0 0" rpy="0 0 0"/>
+            <geometry name="pioneer_geom">
+                <mesh filename="package://p3at_tutorial/meshes/p3at_meshes/top.dae"/>
+            </geometry>
+            <material name="TopBlack">
+                    <color rgba="0.038 0.038 0.038 1.0"/>
+            </material>
+        </visual>
+        <collision>
+            <origin xyz="0 0 0" rpy="0 0 0"/>
+            <geometry>
+                <box size="0.01 0.01 0.01"/>
+            </geometry>
+        </collision>
+    </link>
+    <gazebo reference="top_plate">
+        <material value="Gazebo/Black"/>
+    </gazebo>
+    <joint name="base_top_joint" type="fixed">
+        <origin xyz="0.003 0 0.274" rpy="0 0 0"/>
+        <parent link="base_link"/>
+        <child link="top_plate"/>
+    </joint>
 <!-- Front + Back Sonar -->
-	<link name="front_sonar">
-		<inertial>
-			<mass value="0.1"/>
-			<origin xyz="0 0 0"/>
-			<inertia ixx="1.0" ixy="0.0" ixz="0.0"
-				 iyy="1.0" iyz="0.0" izz="1.0"/>
-		</inertial>
-		<visual name="base_visual">
-			<origin xyz="0 0 0" rpy="0 0 0"/>
-			<geometry name="pioneer_geom">
-				<mesh filename="package://p3at_tutorial/meshes/p3at_meshes/front_sonar.stl"/>
-			</geometry>
-			<material name="SonarYellow">
-				<color rgba="0.715 0.583 0.210 1.0"/>
-			</material>
-		</visual>
-		<collision>
-			<origin xyz="0 0 0" rpy="0 0 0"/>
-			<geometry>
-				<box size="0 0 0"/>
-			</geometry>
-		</collision>
-	</link>
-	<gazebo reference="front_sonar">
-		<material value="Gazebo/Yellow"/>
-	</gazebo>
-	<joint name="base_front_joint" type="fixed">
-		<origin xyz="0.193 0 0.25" rpy="0 0 0"/>
-		<parent link="base_link"/>
-		<child link="front_sonar"/>
-	</joint>
-	<link name="back_sonar">
-		<inertial>
-			<mass value="0.1"/>
-			<origin xyz="0 0 0"/>
-			<inertia ixx="1.0" ixy="0.0" ixz="0.0"
-				 iyy="1.0" iyz="0.0" izz="1.0"/>
-		</inertial>
-		<visual name="base_visual">
-			<origin xyz="0 0 0" rpy="0 0 0"/>
-			<geometry name="pioneer_geom">
-				<mesh filename="package://p3at_tutorial/meshes/p3at_meshes/back_sonar.stl"/>
-			</geometry>
-			<material name="SonarYellow">
-				<color rgba="0.715 0.583 0.210 1.0"/>
-			</material>
-		</visual>
-		<collision>
-			<origin xyz="0 0 0" rpy="0 0 0"/>
-			<geometry>
-				<box size="0 0 0"/>
-			</geometry>
-		</collision>
-	</link>
-	<gazebo reference="back_sonar">
-		<material value="Gazebo/Yellow"/>
-	</gazebo>
-	<joint name="base_back_joint" type="fixed">
-		<origin xyz="-0.187 0 0.247" rpy="0 0 0"/>
-		<parent link="base_link"/>
-		<child link="back_sonar"/>
-	</joint>
-<link name="back_sonar_fake">
-    <inertial>
-            <mass value="0.1"/>
-            <origin xyz="0 0 0"/>
-            <inertia ixx="1.0" ixy="0.0" ixz="0.0"
-                 iyy="1.0" iyz="0.0" izz="1.0"/>
-    </inertial>
-<!--     <visual name="base_visual">
+    <link name="front_sonar">
+        <inertial>
+            <mass value="0.1"/>
+            <origin xyz="0 0 0"/>
+            <inertia ixx="1.0" ixy="0.0" ixz="0.0"
+                 iyy="1.0" iyz="0.0" izz="1.0"/>
+        </inertial>
+        <visual name="base_visual">
             <origin xyz="0 0 0" rpy="0 0 0"/>
             <geometry name="pioneer_geom">
-                <mesh filename="package://p3at_tutorial/meshes/p3at_meshes/back_sonar.stl"/>
+                <mesh filename="package://p3at_tutorial/meshes/p3at_meshes/front_sonar.dae"/>
             </geometry>
             <material name="SonarYellow">
@@ -164,5 +102,67 @@
             <origin xyz="0 0 0" rpy="0 0 0"/>
             <geometry>
-                <box size="0 0 0"/>
+                <box size="0.01 0.01 0.01"/>
+            </geometry>
+        </collision>
+    </link>
+    <gazebo reference="front_sonar">
+        <material value="Gazebo/Yellow"/>
+    </gazebo>
+    <joint name="base_front_joint" type="fixed">
+        <origin xyz="0.193 0 0.25" rpy="0 0 0"/>
+        <parent link="base_link"/>
+        <child link="front_sonar"/>
+    </joint>
+    <link name="back_sonar">
+        <inertial>
+            <mass value="0.1"/>
+            <origin xyz="0 0 0"/>
+            <inertia ixx="1.0" ixy="0.0" ixz="0.0"
+                 iyy="1.0" iyz="0.0" izz="1.0"/>
+        </inertial>
+        <visual name="base_visual">
+            <origin xyz="0 0 0" rpy="0 0 0"/>
+            <geometry name="pioneer_geom">
+                <mesh filename="package://p3at_tutorial/meshes/p3at_meshes/back_sonar.dae"/>
+            </geometry>
+            <material name="SonarYellow">
+                <color rgba="0.715 0.583 0.210 1.0"/>
+            </material>
+        </visual>
+        <collision>
+            <origin xyz="0 0 0" rpy="0 0 0"/>
+            <geometry>
+                <box size="0.01 0.01 0.01"/>
+            </geometry>
+        </collision>
+    </link>
+    <gazebo reference="back_sonar">
+        <material value="Gazebo/Yellow"/>
+    </gazebo>
+    <joint name="base_back_joint" type="fixed">
+        <origin xyz="-0.187 0 0.247" rpy="0 0 0"/>
+        <parent link="base_link"/>
+        <child link="back_sonar"/>
+    </joint>
+<link name="back_sonar_fake">
+    <inertial>
+            <mass value="0.1"/>
+            <origin xyz="0 0 0"/>
+            <inertia ixx="1.0" ixy="0.0" ixz="0.0"
+                 iyy="1.0" iyz="0.0" izz="1.0"/>
+    </inertial>
+<!--     <visual name="base_visual">
+            <origin xyz="0 0 0" rpy="0 0 0"/>
+            <geometry name="pioneer_geom">
+                <mesh filename="package://p3at_tutorial/meshes/p3at_meshes/back_sonar.dae"/>
+            </geometry>
+            <material name="SonarYellow">
+                <color rgba="0.715 0.583 0.210 1.0"/>
+            </material>
+        </visual>
+        <collision>
+            <origin xyz="0 0 0" rpy="0 0 0"/>
+            <geometry>
+                <box size="0.01 0.01 0.01"/>
             </geometry>
         </collision> -->
@@ -183,5 +183,5 @@
             <origin xyz="0 0 0" rpy="0 0 0"/>
             <geometry name="pioneer_geom">
-                <mesh filename="package://p3at_tutorial/meshes/p3at_meshes/back_sonar.stl"/>
+                <mesh filename="package://p3at_tutorial/meshes/p3at_meshes/back_sonar.dae"/>
             </geometry>
             <material name="SonarYellow">
@@ -192,5 +192,5 @@
             <origin xyz="0 0 0" rpy="0 0 0"/>
             <geometry>
-                <box size="0 0 0"/>
+                <box size="0.01 0.01 0.01"/>
             </geometry>
         </collision> -->
@@ -203,203 +203,203 @@
 <!-- Front Axles + Wheels + Hubcaps -->
 <xacro:macro name="p3at_front" params="suffix reflect">
-	<link name="p3at_front_${suffix}_axle">
-		<inertial>
-			<mass value="0.1"/>
-			<origin xyz="0 0 0"/>
-			<inertia ixx="1.0" ixy="0.0" ixz="0.0"
-				 iyy="1.0" iyz="0.0" izz="1.0"/>
-  	 	</inertial>
-	<visual name="base_visual">
-		<origin xyz="0 0 0" rpy="0 0 0"/>
-		<geometry name="pioneer_geom">
-			<mesh filename="package://p3at_tutorial/meshes/p3at_meshes/axle.stl"/>
-		</geometry>
-		<material name="AxleGrey">
-			<color rgba="0.5 0.5 0.5 1"/>
-		</material>
-	</visual>
-	<collision>
-		<origin xyz="0 0 0" rpy="0 0 0"/>
-		<geometry>
-			<box size="0 0 0"/>
-		</geometry>
-	</collision>
-	</link>
-	<gazebo reference="p3at_front_${suffix}_axle">
-		<material value="Gazebo/Grey"/>
-	</gazebo>
-	<joint name="base_front_${suffix}_axle_joint" type="fixed">
-		<origin xyz="0.135 ${reflect*0.156} 0.111" rpy="0 0 0"/>
-		<parent link="base_link"/>
-		<child link="p3at_front_${suffix}_axle"/>
-	</joint>
-	<link name="p3at_front_${suffix}_hub">
-		<inertial>
-			<mass value="0.1"/>
-			<origin xyz="0 0 0"/>
-			<inertia ixx="1.0" ixy="0.0" ixz="0.0"
-				 iyy="1.0" iyz="0.0" izz="1.0"/>
-  	 	</inertial>
-	<visual name="base_visual">
-		<origin xyz="0 0 0" rpy="0 0 0"/>
-		<geometry name="pioneer_geom">
-			<mesh filename="package://p3at_tutorial/meshes/p3at_meshes/${suffix}_hubcap.stl"/>
-		</geometry>
-		<material name="HubcapYellow">
-			<color rgba="1.0 0.811 0.151 1.0"/>
-		</material>
-	</visual>
-	<collision>
-		<origin xyz="0 0 0" rpy="0 0 0"/>
-		<geometry>
-			<box size="0 0 0"/>
-		</geometry>
-	</collision>
-	</link>
-	<gazebo reference="p3at_front_${suffix}_hub">
-		<material value="Gazebo/Yellow"/>
-	</gazebo>
-	<joint name="base_front_${suffix}_hub_joint" type="fixed">
-		<origin xyz="0 ${reflect*0.041} 0" rpy="0 0 0"/>
-		<parent link="p3at_front_${suffix}_axle"/>
-		<child link="p3at_front_${suffix}_hub"/>
-	</joint>
-	<link name="p3at_front_${suffix}_wheel">
-		<inertial>
-			<mass value="0.5"/>
-			<origin xyz="0 0 0"/>
-			<inertia ixx="0.012411765597" ixy="0" ixz="0"
+    <link name="p3at_front_${suffix}_axle">
+        <inertial>
+            <mass value="0.1"/>
+            <origin xyz="0 0 0"/>
+            <inertia ixx="1.0" ixy="0.0" ixz="0.0"
+                 iyy="1.0" iyz="0.0" izz="1.0"/>
+        </inertial>
+    <visual name="base_visual">
+        <origin xyz="0 0 0" rpy="0 0 0"/>
+        <geometry name="pioneer_geom">
+            <mesh filename="package://p3at_tutorial/meshes/p3at_meshes/axle.dae"/>
+        </geometry>
+        <material name="AxleGrey">
+            <color rgba="0.5 0.5 0.5 1"/>
+        </material>
+    </visual>
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